File: PCB.kicad_pcb (KiCad board)
At the start: 2 copper layers, 15 parts, among them J1 Conector alimentacao servo, J11 Servo, J12 IR1, J13 IR2, J14 Conector LORA, J15 Conector motor esquerdo, J16 Conector motor direito, J17 Conector ultrassonico, J18 LEDs, J2 Conector bluetooth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

Commit message: feat: criacao do pcb
Parts:
- removed J1: Conector alimentacao servo, TerminalBlock_Phoenix:TerminalBlock_Phoenix_MKDS-1,5-2_1x02_P5.00mm_Horizontal
- removed J11: Servo, Connector_PinHeader_2.54mm:PinHeader_1x01_P2.54mm_Vertical
- removed J12: IR1, Connector_PinHeader_2.54mm:PinHeader_1x01_P2.54mm_Vertical
- removed J13: IR2, Connector_PinHeader_2.54mm:PinHeader_1x01_P2.54mm_Vertical
- removed J15: Conector motor esquerdo, Connector_PinSocket_2.54mm:PinSocket_2x03_P2.54mm_Vertical
- removed J16: Conector motor direito, Connector_PinSocket_2.54mm:PinSocket_2x03_P2.54mm_Vertical
- removed J17: Conector ultrassonico, Connector_PinSocket_2.54mm:PinSocket_2x06_P2.54mm_Vertical
- added +5V SENSORES: Conector alimentacao sensores, TerminalBlock_Phoenix:TerminalBlock_Phoenix_MKDS-1,5-2_1x02_P5.00mm_Horizontal, F.Cu at (139.6, 157.5)
- added INFRAVERMELHO: Conector IR, Connector_JST:JST_XH_B2B-XH-A_1x02_P2.50mm_Vertical, F.Cu at (71.0, 114.3)
- added J7: PONTA H 1, Connector_PinSocket_2.54mm:PinSocket_2x04_P2.54mm_Vertical, B.Cu at (63.4, 152.4)
- added LED EXTRA: Conector LED Extra, Connector_JST:JST_XH_B2B-XH-A_1x02_P2.50mm_Vertical, F.Cu at (142.1, 142.2)
- added PONTE H 2: Conector motor esquerdo, Connector_PinSocket_2.54mm:PinSocket_2x04_P2.54mm_Vertical, B.Cu at (129.4, 152.4)
- added R1: R, Resistor_THT:R_Axial_DIN0207_L6.3mm_D2.5mm_P10.16mm_Horizontal, F.Cu at (139.6, 147.3)
- added REF**: MountingHole_3.2mm_M3, MountingHole:MountingHole_3.2mm_M3, F.Cu at (170.1, 40.6)
- added REF**: MountingHole_3.2mm_M3, MountingHole:MountingHole_3.2mm_M3, F.Cu at (50.7, 40.6)
- added REF**: MountingHole_3.2mm_M3, MountingHole:MountingHole_3.2mm_M3, F.Cu at (124.3, 142.2)
- added REF**: MountingHole_3.2mm_M3, MountingHole:MountingHole_3.2mm_M3, F.Cu at (58.3, 142.2)
- added ULTRASSONICO CEN: Conector ultrassonico central, Connector_JST:JST_XH_B4B-XH-A_1x04_P2.50mm_Vertical, F.Cu at (142.1, 121.9)
- added ULTRASSONICO DIR: Conector ultrassonico direito, Connector_JST:JST_XH_B4B-XH-A_1x04_P2.50mm_Vertical, F.Cu at (142.1, 132.1)
- added ULTRASSONICO ESQ: Conector ultrassonico esquerdo, Connector_JST:JST_XH_B4B-XH-A_1x04_P2.50mm_Vertical, F.Cu at (142.1, 111.8)
- ENCO DIR: renamed from J6
- ENCO ESQ: renamed from J4
- LORA: renamed from J14; footprint TerminalBlock_Phoenix:TerminalBlock_Phoenix_MKDS-1,5-4_1x04_P5.00mm_Horizontal -> Connector_JST:JST_XH_B4B-XH-A_1x04_P2.50mm_Vertical
- SERVO: renamed from J5; value HC6 -> Conector servo; footprint Connector_PinSocket_2.54mm:PinSocket_1x02_P2.54mm_Vertical -> TerminalBlock_Phoenix:TerminalBlock_Phoenix_MKDS-1,5-3_1x03_P5.00mm_Horizontal
- XA1: footprint PCM_arduino-library:Arduino_Mega2560_R3_Shield -> PCM_arduino-library:Arduino_Mega2560_R3_Shield_Sem_furo
- moved SERVO 115.7 mm to (96.5, 155.2)
- moved ENCO DIR 113.9 mm to (83.7, 154.9)
- moved ENCO ESQ 111.5 mm to (71.0, 154.9)
- moved BLUETOOTH 92.6 mm to (116.7, 116.8)
- moved XA1 69.5 mm to (43.1, 104.1)
- moved LORA 68.6 mm to (78.6, 127.0), turned to 180 degrees
- moved LEDs 60.8 mm to (58.0, 114.5)
- moved ACELEROMETRO 32.6 mm to (101.5, 111.8), turned to 0 degrees
- renumbered J3 to ACELEROMETRO, J2 to BLUETOOTH, J18 to LEDs
Connections:
- SERVO pad 1: Net-(J5-Pin_1) -> Servo
- SERVO pad 2: Net-(J5-Pin_2) -> 5V_Sen
- XA1 pad D30: Net-(J12-Pin_1) -> IR1
- XA1 pad D36: unconnected-(XA1-PadD36) -> LED_Extra
- XA1 pad D46: Net-(J13-Pin_1) -> IR2
- XA1 pad D50: Net-(J5-Pin_2) -> HC6_1
- XA1 pad D51: Net-(J5-Pin_1) -> HC6_2
- XA1 pad D8: Net-(J11-Pin_1) -> Servo
Routing:
- net Earth: track 0.00 -> 363.2 mm, vias 0 -> 6
- net ME2: track 0.00 -> 266.5 mm, vias 0 -> 3
- net Servo: track 0.00 -> 256.7 mm, vias 0 -> 2
- net ME1: track 0.00 -> 252.0 mm, vias 0 -> 3
- net 5V_Sen: track 0.00 -> 231.0 mm, vias 0 -> 2
- net Net-(J6-Pin_2): track 0.00 -> 213.2 mm, vias 0 -> 3
- net LED_Extra: track 0.00 -> 203.8 mm, vias 0 -> 6
- net Net-(J18-Pin_3): track 0.00 -> 202.2 mm, vias 0 -> 2
- net ECHO_1: track 0.00 -> 189.7 mm, vias 0 -> 3
- net TRIG_1: track 0.00 -> 186.5 mm, vias 0 -> 2
- net Net-(J18-Pin_1): track 0.00 -> 178.8 mm
- net Net-(J4-Pin_2): track 0.00 -> 169.8 mm, vias 0 -> 6
- net Net-(J4-Pin_1): track 0.00 -> 165.0 mm, vias 0 -> 4
- net TRIG_3: track 0.00 -> 163.0 mm, vias 0 -> 4
- net Net-(J18-Pin_4): track 0.00 -> 155.5 mm, vias 0 -> 6
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- added copper zone on B.Cu, net Earth
Other:
- board outline added: 147.3 x 142.2 mm
- board text added: "+5V"
- board text added: "D18"
- board text added: "D19"
- board text added: "D2"
- board text added: "D3"
- board text added: "FAROIS"
- board text added: "FREIOS"
- board text added: "GND"
- board text added: "SERVO"
- board text added: "SETA DIR"
- board text added: "SETA ESQ"
