File: PCB.kicad_sch (KiCad schematic)
At the start: 15 parts, among them J1 Conector alimentacao servo, J11 Servo, J12 IR1, J13 IR2, J14 Conector LORA, J15 Conector motor esquerdo, J16 Conector motor direito, J17 Conector ultrassonico, J18 LEDs, J2 Conector bluetooth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

Commit message: feat: criacao do pcb
Parts:
- removed J11: Servo, Connector_PinHeader_2.54mm:PinHeader_1x01_P2.54mm_Vertical, symbol Connector:Conn_01x01_Pin
- removed J12: IR1, Connector_PinHeader_2.54mm:PinHeader_1x01_P2.54mm_Vertical, symbol Connector:Conn_01x01_Pin
- removed J13: IR2, Connector_PinHeader_2.54mm:PinHeader_1x01_P2.54mm_Vertical, symbol Connector:Conn_01x01_Pin
- removed J15: Conector motor esquerdo, Connector_PinSocket_2.54mm:PinSocket_2x03_P2.54mm_Vertical, symbol Connector:Conn_01x06_Pin
- removed J16: Conector motor direito, Connector_PinSocket_2.54mm:PinSocket_2x03_P2.54mm_Vertical, symbol Connector:Conn_01x06_Pin
- removed J17: Conector ultrassonico, Connector_PinSocket_2.54mm:PinSocket_2x06_P2.54mm_Vertical, symbol Connector:Conn_01x12_Pin
- removed J5: HC6, Connector_PinSocket_2.54mm:PinSocket_1x02_P2.54mm_Vertical, symbol Connector:Conn_01x02_Pin
- added J10: Conector ultrassonico esquerdo, Connector_JST:JST_XH_B4B-XH-A_1x04_P2.50mm_Vertical, symbol Connector:Conn_01x04_Pin
- added J11: Conector ultrassonico central, Connector_JST:JST_XH_B4B-XH-A_1x04_P2.50mm_Vertical, symbol Connector:Conn_01x04_Pin
- added J12: Conector ultrassonico direito, Connector_JST:JST_XH_B4B-XH-A_1x04_P2.50mm_Vertical, symbol Connector:Conn_01x04_Pin
- added J13: Conector LED Extra, Connector_JST:JST_XH_B2B-XH-A_1x02_P2.50mm_Vertical, symbol Connector:Conn_01x02_Pin
- added J5: Conector servo, TerminalBlock_Phoenix:TerminalBlock_Phoenix_MKDS-1,5-3_1x03_P5.00mm_Horizontal, symbol Connector:Conn_01x03_Pin
- added J7: Conector motor direito, Connector_PinSocket_2.54mm:PinSocket_2x04_P2.54mm_Vertical, symbol Connector:Conn_01x08_Pin
- added J8: Conector motor esquerdo, Connector_PinSocket_2.54mm:PinSocket_2x04_P2.54mm_Vertical, symbol Connector:Conn_01x08_Pin
- added J9: Conector alimentacao sensores, TerminalBlock_Phoenix:TerminalBlock_Phoenix_MKDS-1,5-2_1x02_P5.00mm_Horizontal, symbol Connector:Conn_01x02_Pin
- added R1: R, Resistor_THT:R_Axial_DIN0207_L6.3mm_D2.5mm_P10.16mm_Horizontal, symbol Device:R
- J1: value Conector alimentacao servo -> Conector IR; footprint TerminalBlock_Phoenix:TerminalBlock_Phoenix_MKDS-1,5-2_1x02_P5.00mm_Horizontal -> Connector_JST:JST_XH_B2B-XH-A_1x02_P2.50mm_Vertical
- J14: footprint TerminalBlock_Phoenix:TerminalBlock_Phoenix_MKDS-1,5-4_1x04_P5.00mm_Horizontal -> Connector_JST:JST_XH_B4B-XH-A_1x04_P2.50mm_Vertical
- XA1: footprint PCM_arduino-library:Arduino_Mega2560_R3_Shield -> PCM_arduino-library:Arduino_Mega2560_R3_Shield_Sem_furo
Connections:
- net 5V_Sen: now also J10.1 (Pin_1), J11.1 (Pin_1), J12.1 (Pin_1), J5.2 (Pin_2), J7.1 (Pin_1), J7.3 (Pin_3), J7.4 (Pin_4), J8.1 (Pin_1), J8.3 (Pin_3), J8.4 (Pin_4), J9.1 (Pin_1); no longer J1.1 (Pin_1)
- net ECHO_1: now also J10.2 (Pin_2)
- net ECHO_2: now also J11.2 (Pin_2)
- net ECHO_3: now also J12.2 (Pin_2)
- net Earth: now also J10.4 (Pin_4), J11.4 (Pin_4), J12.4 (Pin_4), J13.2 (Pin_2), J5.3 (Pin_3), J7.2 (Pin_2), J8.2 (Pin_2), J9.2 (Pin_2); no longer J1.2 (Pin_2)
- net HC6_1: now also XA1.D50 (D50_MISO)
- net HC6_2: now also XA1.D51 (D51_MOSI)
- net MD1: now also J7.8 (Pin_8)
- net MD2: now also J7.7 (Pin_7)
- net ME1: now also J8.8 (Pin_8)
- net ME2: now also J8.7 (Pin_7)
- net TRIG_1: now also J10.3 (Pin_3)
- net TRIG_2: now also J11.3 (Pin_3)
- net TRIG_3: now also J12.3 (Pin_3)
- net IR1: now reaches XA1.D30
- net IR1: now also J1.1 (Pin_1)
- net LED_Extra: now reaches XA1.D36
- net LED_Extra: now also R1.2
- net IR2: now reaches XA1.D46
- net IR2: now also J1.2 (Pin_2)
- net Servo: now reaches XA1.D8
- net Servo: now also J5.1 (Pin_1)
- new net: J13.1 (Pin_1), R1.1

Commit message: feat: inicio da nova versao da pcb
Parts:
- removed J4: ENCO_SW_Esq, TerminalBlock_Phoenix:TerminalBlock_Phoenix_MKDS-1,5-2_1x02_P5.00mm_Horizontal, symbol Connector:Conn_01x02_Pin
- removed J6: ENCO_SW_Dir, TerminalBlock_Phoenix:TerminalBlock_Phoenix_MKDS-1,5-2_1x02_P5.00mm_Horizontal, symbol Connector:Conn_01x02_Pin
- added J15: ENCO_SW_Esq, TerminalBlock_Phoenix:TerminalBlock_Phoenix_MKDS-1,5-4_1x04_P5.00mm_Horizontal, symbol Connector:Conn_01x04_Pin
- added J16: ENCO_SW_Dir, TerminalBlock_Phoenix:TerminalBlock_Phoenix_MKDS-1,5-4_1x04_P5.00mm_Horizontal, symbol Connector:Conn_01x04_Pin
Connections:
- net 5V_Sen: now also J15.1 (Pin_1), J16.1 (Pin_1)
- net Earth: now also J15.4 (Pin_4), J16.4 (Pin_4)
- net ENCODER_Dir_1: now reaches XA1.D18 (D18/TX1)
- net ENCODER_Dir_1: now also J15.2 (Pin_2)
- net ENCODER_Dir_2: now reaches XA1.D19 (D19/RX1)
- net ENCODER_Dir_2: now also J15.3 (Pin_3)
- net ENCODER_Esq_1: now reaches XA1.D2 (D2_INT0)
- net ENCODER_Esq_1: now also J16.2 (Pin_2)
- net ENCODER_Esq_2: now reaches XA1.D3 (D3_INT1)
- net ENCODER_Esq_2: now also J16.3 (Pin_3)

Commit message: feat: finalizacao da versao 2 da pcb
Connections:
- net 5V_Sen: now also J7.2 (Pin_2), J8.2 (Pin_2); no longer J7.1 (Pin_1), J8.1 (Pin_1)
- net Earth: now also J7.1 (Pin_1), J8.1 (Pin_1); no longer J7.2 (Pin_2), J8.2 (Pin_2)
Changed lines of the file:
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@@
 (kicad_sch (version 20230121) (generator eeschema)
   (paper "A4")
+  (wire (pts (xy 77.47 168.91) (xy 90.17 168.91))
+    (stroke (width 0) (type default))
+  )
   (wire (pts (xy 48.26 152.4) (xy 49.53 152.4))
     (stroke (width 0) (type default))
@@
     (stroke (width 0) (type default))
   )
-  (wire (pts (xy 90.17 171.45) (xy 90.17 172.72))
-    (stroke (width 0) (type default))
-  )
   (wire (pts (xy 193.04 146.05) (xy 194.31 146.05))
     (stroke (width 0) (type default))
@@
     (stroke (width 0) (type default))
   )
+  (wire (pts (xy 90.17 168.91) (xy 90.17 170.18))
+    (stroke (width 0) (type default))
+  )
+  (wire (pts (xy 55.88 168.91) (xy 55.88 170.18))
+    (stroke (width 0) (type default))
+  )
   (wire (pts (xy 138.43 166.37) (xy 152.4 166.37))
     (stroke (width 0) (type default))
@@
     (stroke (width 0) (type default))
   )
-  (wire (pts (xy 77.47 171.45) (xy 90.17 171.45))
+  (wire (pts (xy 43.18 168.91) (xy 55.88 168.91))
     (stroke (width 0) (type default))
   )
@@
     (stroke (width 0) (type default))
   )
-  (wire (pts (xy 43.18 171.45) (xy 55.88 171.45))
-    (stroke (width 0) (type default))
-  )
   (wire (pts (xy 166.37 158.75) (xy 167.64 158.75))
     (stroke (width 0) (type default))
   )
   (wire (pts (xy 111.76 176.53) (xy 111.76 177.8))
-    (stroke (width 0) (type default))
-  )
-  (wire (pts (xy 55.88 171.45) (xy 55.88 172.72))
     (stroke (width 0) (type default))
   )
@@
     )
   )
-  (global_label "5V_Sen" (shape bidirectional) (at 77.47 168.91 0) (fields_autoplaced)
-    (effects (font (size 1.27 1.27)) (justify left))
-    (property "Intersheetrefs" "${INTERSHEET_REFS}" (at 88.2793 168.91 0)
-      (effects (font (size 1.27 1.27)) (justify left) hide)
-    )
-  )
   (global_label "ECHO_2" (shape bidirectional) (at 138.43 161.29 0) (fields_autoplaced)
     (effects (font (size 1.27 1.27)) (justify left))
@@
     )
   )
-  (global_label "5V_Sen" (shape bidirectional) (at 43.18 168.91 0) (fields_autoplaced)
-    (effects (font (size 1.27 1.27)) (justify left))
-    (property "Intersheetrefs" "${INTERSHEET_REFS}" (at 53.9893 168.91 0)
+  (global_label "5V_Sen" (shape bidirectional) (at 43.18 171.45 0) (fields_autoplaced)
+    (effects (font (size 1.27 1.27)) (justify left))
+    (property "Intersheetrefs" "${INTERSHEET_REFS}" (at 53.9893 171.45 0)
       (effects (font (size 1.27 1.27)) (justify left) hide)
     )
@@
     (effects (font (size 1.27 1.27)) (justify left))
     (property "Intersheetrefs" "${INTERSHEET_REFS}" (at 148.816 144.78 0)
+      (effects (font (size 1.27 1.27)) (justify left) hide)
+    )
+  )
+  (global_label "5V_Sen" (shape bidirectional) (at 77.47 171.45 0) (fields_autoplaced)
+    (effects (font (size 1.27 1.27)) (justify left))
+    (property "Intersheetrefs" "${INTERSHEET_REFS}" (at 88.2793 171.45 0)
       (effects (font (size 1.27 1.27)) (justify left) hide)
     )
@@
     )
   )
+  (symbol (lib_id "power:Earth") (at 90.17 170.18 0) (unit 1)
+    (in_bom yes) (on_board yes) (dnp no) (fields_autoplaced)
+    (property "Reference" "#PWR04" (at 90.17 176.53 0)
+      (effects (font (size 1.27 1.27)) hide)
+    )
+    (property "Value" "Earth" (at 90.17 173.99 0)
+      (effects (font (size 1.27 1.27)) hide)
+    )
+    (property "Footprint" "" (at 90.17 170.18 0)
+      (effects (font (size 1.27 1.27)) hide)
+    )
+    (property "Datasheet" "~" (at 90.17 170.18 0)
+      (effects (font (size 1.27 1.27)) hide)
+    )
+    (pin "1")
+    (instances
+      (project "PCB"
+        (path "/b344186f-9059-49c5-a6f7-f90c862ad97f"
+          (reference "#PWR04") (unit 1)
+        )
+      )
+      (project "esquemaEletricoCarro"
+        (path "/e63e39d7-6ac0-4ffd-8aa3-1841a4541b55/980d7ea7-3ff9-498b-b91b-57f4a8ccee38"
+          (reference "#PWR08") (unit 1)
+        )
+      )
+    )
+  )
   (symbol (lib_id "Device:R") (at 203.2 143.51 90) (unit 1)
     (in_bom yes) (on_board yes) (dnp no) (fields_autoplaced)
@@
         (path "/e63e39d7-6ac0-4ffd-8aa3-1841a4541b55/ef1da815-5ae9-4f7a-859c-d7960e6acc1e"
           (reference "#PWR021") (unit 1)
-        )
-      )
-    )
-  )
-  (symbol (lib_id "power:Earth") (at 90.17 172.72 0) (unit 1)
-    (in_bom yes) (on_board yes) (dnp no) (fields_autoplaced)
-    (property "Reference" "#PWR04" (at 90.17 179.07 0)
-      (effects (font (size 1.27 1.27)) hide)
-    )
-    (property "Value" "Earth" (at 90.17 176.53 0)
-      (effects (font (size 1.27 1.27)) hide)
-    )
-    (property "Footprint" "" (at 90.17 172.72 0)
-      (effects (font (size 1.27 1.27)) hide)
-    )
-    (property "Datasheet" "~" (at 90.17 172.72 0)
-      (effects (font (size 1.27 1.27)) hide)
-    )
-    (pin "1")
-    (instances
-      (project "PCB"
-        (path "/b344186f-9059-49c5-a6f7-f90c862ad97f"
-          (reference "#PWR04") (unit 1)
-        )
-      )
-      (project "esquemaEletricoCarro"
-        (path "/e63e39d7-6ac0-4ffd-8aa3-1841a4541b55/980d7ea7-3ff9-498b-b91b-57f4a8ccee38"
-          (reference "#PWR08") (unit 1)
         )
       )
@@
     )
   )
-  (symbol (lib_id "power:Earth") (at 55.88 172.72 0) (unit 1)
-    (in_bom yes) (on_board yes) (dnp no) (fields_autoplaced)
-    (property "Reference" "#PWR010" (at 55.88 179.07 0)
-      (effects (font (size 1.27 1.27)) hide)
-    )
-    (property "Value" "Earth" (at 55.88 176.53 0)
-      (effects (font (size 1.27 1.27)) hide)
-    )
-    (property "Footprint" "" (at 55.88 172.72 0)
-      (effects (font (size 1.27 1.27)) hide)
-    )
-    (property "Datasheet" "~" (at 55.88 172.72 0)
-      (effects (font (size 1.27 1.27)) hide)
-    )
+  (symbol (lib_id "power:Earth") (at 55.88 170.18 0) (unit 1)
+    (in_bom yes) (on_board yes) (dnp no) (fields_autoplaced)
+    (property "Reference" "#PWR010" (at 55.88 176.53 0)
+      (effects (font (size 1.27 1.27)) hide)
+    )
+    (property "Value" "Earth" (at 55.88 173.99 0)
+      (effects (font (size 1.27 1.27)) hide)
+    )
+    (property "Footprint" "" (at 55.88 170.18 0)
+      (effects (font (size 1.27 1.27)) hide)
+    )
+    (property "Datasheet" "~" (at 55.88 170.18 0)
+      (effects (font (size 1.27 1.27)) hide)
+    )
