File: V3/PCB V3.kicad_pcb (KiCad board)
At the start: 2 copper layers, 97.5 x 128.5 mm, 26 parts, among them J1 Conector motor esquerdo, J10 Conector LORA, J11 Conector ultrassonico esquerdo, J12 Conector ultrassonico central, J13 Conector ultrassonico direito, J14 Conector IR esquerdo, J15 Conector IR direito, J16 Conector LED Faróis, J17 Conector LED Extra, J2 Conector motor direito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

Commit message: feat: criação dos arquivos de manufatura
Parts:
- moved G*** 78.3 mm to (129.7, 76.8), turned to 90 degrees
- moved J4 12.9 mm to (110.3, 124.2)
- moved J5 12.9 mm to (183.4, 65.1)
- moved J7 12.9 mm to (110.3, 86.1)
- moved J9 12.9 mm to (186.3, 106.8)
- moved REF** 12.9 mm to (110.3, 139.8)
- moved XA1 12.9 mm to (172.8, 146.9)
- moved G*** 12.9 mm to (165.7, 62.1)
- moved J12 12.9 mm to (128.5, 33.0)
- moved J13 12.9 mm to (136.0, 33.0)
- moved J14 12.9 mm to (185.5, 54.0)
- moved J15 12.9 mm to (185.5, 46.8)
- moved J16 12.9 mm to (178.8, 35.1)
- moved J17 12.9 mm to (147.2, 33.0)
- moved J6 12.9 mm to (110.3, 50.5)
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Routing:
- net MD1: track 85.7 -> 88.8 mm
- net MD2: track 81.4 -> 84.6 mm
- net 5V_Sen: vias 5 -> 4
- net HC6_1: vias 5 -> 4
Other:
- outline, holes or cut-outs redrawn
- board text removed: "09 de Setembro de 2023 | Autonomous Vehicles Challenge"
